File: Connectors.kicad_sch (KiCad schematic)
At the start: 2 parts

Commit message: WIP update
Parts:
- gave numbers to parts that had none: 2
Other:
- note added: "Connectors"
- moved on the sheet: J1, U2

Commit message: WIP update
Other:
- moved on the sheet: J1, U2
