File: POWER.kicad_sch (KiCad schematic)
At the start: 1 part

Commit message: WIP update
Parts:
- added C1, C2: 10u, symbol Device:C_Small
- added F1: Fuse, symbol Device:Fuse
- added FB1: 100@100MHz, symbol Device:FerriteBead
- gave numbers to parts that had none: 1
Connections:
- net GND: now reaches U3.1 (GND)
- net GND: now also C1.2, C2.2
- net +3.3V: now reaches U3.2 (VO)
- net +3.3V: now also C2.1
- net at U3.3 (VI): now also C1.1, FB1.2
- new net: F1.2, FB1.1
- new net +5V: F1.1
Other:
- note added: "POWER"
- moved on the sheet: U3
Changed lines of the file:
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@@
 (kicad_sch (version 20211123) (generator eeschema)
   (paper "A4")
-  (symbol (lib_id "Regulator_Linear:XC6206PxxxMR") (at 81.28 55.88 0) (unit 1)
+  (junction (at 148.59 105.41) (diameter 0) (color 0 0 0 0)
+  )
+  (junction (at 138.43 93.98) (diameter 0) (color 0 0 0 0)
+  )
+  (junction (at 160.02 93.98) (diameter 0) (color 0 0 0 0)
+  )
+  (wire (pts (xy 148.59 101.6) (xy 148.59 105.41))
+    (stroke (width 0) (type default) (color 0 0 0 0))
+  )
+  (wire (pts (xy 138.43 93.98) (xy 140.97 93.98))
+    (stroke (width 0) (type default) (color 0 0 0 0))
+  )
+  (wire (pts (xy 148.59 105.41) (xy 160.02 105.41))
+    (stroke (width 0) (type default) (color 0 0 0 0))
+  )
+  (wire (pts (xy 138.43 93.98) (xy 138.43 97.79))
+    (stroke (width 0) (type default) (color 0 0 0 0))
+  )
+  (wire (pts (xy 156.21 93.98) (xy 160.02 93.98))
+    (stroke (width 0) (type default) (color 0 0 0 0))
+  )
+  (wire (pts (xy 160.02 105.41) (xy 160.02 102.87))
+    (stroke (width 0) (type default) (color 0 0 0 0))
+  )
+  (wire (pts (xy 138.43 105.41) (xy 148.59 105.41))
+    (stroke (width 0) (type default) (color 0 0 0 0))
+  )
+  (wire (pts (xy 109.22 93.98) (xy 114.3 93.98))
+    (stroke (width 0) (type default) (color 0 0 0 0))
+  )
+  (wire (pts (xy 121.92 93.98) (xy 127 93.98))
+    (stroke (width 0) (type default) (color 0 0 0 0))
+  )
+  (wire (pts (xy 163.83 93.98) (xy 160.02 93.98))
+    (stroke (width 0) (type default) (color 0 0 0 0))
+  )
+  (wire (pts (xy 163.83 90.17) (xy 163.83 93.98))
+    (stroke (width 0) (type default) (color 0 0 0 0))
+  )
+  (wire (pts (xy 109.22 91.44) (xy 109.22 93.98))
+    (stroke (width 0) (type default) (color 0 0 0 0))
+  )
+  (wire (pts (xy 160.02 93.98) (xy 160.02 97.79))
+    (stroke (width 0) (type default) (color 0 0 0 0))
+  )
+  (wire (pts (xy 134.62 93.98) (xy 138.43 93.98))
+    (stroke (width 0) (type default) (color 0 0 0 0))
+  )
+  (wire (pts (xy 148.59 105.41) (xy 148.59 106.68))
+    (stroke (width 0) (type default) (color 0 0 0 0))
+  )
+  (wire (pts (xy 138.43 105.41) (xy 138.43 102.87))
+    (stroke (width 0) (type default) (color 0 0 0 0))
+  )
+  (text "POWER\n" (at 24.13 22.86 0)
+    (effects (font (size 4 4) (thickness 0.8) bold) (justify left bottom))
+  )
+  (symbol (lib_id "Regulator_Linear:XC6206PxxxMR") (at 148.59 93.98 0) (unit 1)
     (in_bom yes) (on_board yes) (fields_autoplaced)
-    (property "Reference" "U?" (id 0) (at 81.28 50.2752 0))
-    (property "Value" "XC6206PxxxMR" (id 1) (at 81.28 52.8121 0))
-    (property "Footprint" "Package_TO_SOT_SMD:SOT-23" (id 2) (at 81.28 50.165 0)
+    (property "Reference" "U3" (id 0) (at 148.59 88.3752 0))
+    (property "Value" "XC6206PxxxMR" (id 1) (at 148.59 90.9121 0))
+    (property "Footprint" "Package_TO_SOT_SMD:SOT-23" (id 2) (at 148.59 88.265 0)
       (effects (font (size 1.27 1.27) italic) hide)
     )
-    (property "Datasheet" "https://www.torexsemi.com/file/xc6206/XC6206.pdf" (id 3) (at 81.28 55.88 0)
+    (property "Datasheet" "https://www.torexsemi.com/file/xc6206/XC6206.pdf" (id 3) (at 148.59 93.98 0)
       (effects (font (size 1.27 1.27)) hide)
     )
@@
     (pin "3")
   )
+  (symbol (lib_id "Device:C_Small") (at 160.02 100.33 0) (unit 1)
+    (in_bom yes) (on_board yes) (fields_autoplaced)
+    (property "Reference" "C2" (id 0) (at 162.3441 99.5016 0)
+      (effects (font (size 1.27 1.27)) (justify left))
+    )
+    (property "Value" "10u" (id 1) (at 162.3441 102.0385 0)
+      (effects (font (size 1.27 1.27)) (justify left))
+    )
+    (property "Footprint" "" (id 2) (at 160.02 100.33 0)
+      (effects (font (size 1.27 1.27)) hide)
+    )
+    (property "Datasheet" "~" (id 3) (at 160.02 100.33 0)
+      (effects (font (size 1.27 1.27)) hide)
+    )
+    (pin "1")
+    (pin "2")
+  )
+  (symbol (lib_id "Device:Fuse") (at 118.11 93.98 90) (unit 1)
+    (in_bom yes) (on_board yes) (fields_autoplaced)
+    (property "Reference" "F1" (id 0) (at 118.11 89.5182 90))
+    (property "Value" "Fuse" (id 1) (at 118.11 92.0551 90))
+    (property "Footprint" "" (id 2) (at 118.11 95.758 90)
+      (effects (font (size 1.27 1.27)) hide)
+    )
+    (property "Datasheet" "~" (id 3) (at 118.11 93.98 0)
+      (effects (font (size 1.27 1.27)) hide)
+    )
+    (pin "1")
+    (pin "2")
+  )
+  (symbol (lib_id "power:+3.3V") (at 163.83 90.17 0) (unit 1)
+    (in_bom yes) (on_board yes) (fields_autoplaced)
+    (property "Reference" "#PWR07" (id 0) (at 163.83 93.98 0)
+      (effects (font (size 1.27 1.27)) hide)
+    )
+    (property "Value" "+3.3V" (id 1) (at 163.83 86.5942 0))
+    (property "Footprint" "" (id 2) (at 163.83 90.17 0)
+      (effects (font (size 1.27 1.27)) hide)
+    )
+    (property "Datasheet" "" (id 3) (at 163.83 90.17 0)
+      (effects (font (size 1.27 1.27)) hide)
+    )
+    (pin "1")
+  )
+  (symbol (lib_id "power:+5V") (at 109.22 91.44 0) (unit 1)
+    (in_bom yes) (on_board yes) (fields_autoplaced)
+    (property "Reference" "#PWR05" (id 0) (at 109.22 95.25 0)
+      (effects (font (size 1.27 1.27)) hide)
+    )
+    (property "Value" "+5V" (id 1) (at 109.22 87.8642 0))
+    (property "Footprint" "" (id 2) (at 109.22 91.44 0)
+      (effects (font (size 1.27 1.27)) hide)
+    )
+    (property "Datasheet" "" (id 3) (at 109.22 91.44 0)
+      (effects (font (size 1.27 1.27)) hide)
+    )
+    (pin "1")
+  )
+  (symbol (lib_id "power:GND") (at 148.59 106.68 0) (unit 1)
+    (in_bom yes) (on_board yes) (fields_autoplaced)
+    (property "Reference" "#PWR06" (id 0) (at 148.59 113.03 0)
+      (effects (font (size 1.27 1.27)) hide)
+    )
+    (property "Value" "GND" (id 1) (at 148.59 111.1234 0))
+    (property "Footprint" "" (id 2) (at 148.59 106.68 0)
+      (effects (font (size 1.27 1.27)) hide)
+    )
+    (property "Datasheet" "" (id 3) (at 148.59 106.68 0)
+      (effects (font (size 1.27 1.27)) hide)
+    )
+    (pin "1")
+  )
+  (symbol (lib_id "Device:FerriteBead") (at 130.81 93.98 90) (unit 1)
+    (in_bom yes) (on_board yes) (fields_autoplaced)
+    (property "Reference" "FB1" (id 0) (at 130.7592 87.6386 90))
+    (property "Value" "100@100MHz" (id 1) (at 130.7592 90.1755 90))
+    (property "Footprint" "" (id 2) (at 130.81 95.758 90)
+      (effects (font (size 1.27 1.27)) hide)
+    )
+    (property "Datasheet" "~" (id 3) (at 130.81 93.98 0)
+      (effects (font (size 1.27 1.27)) hide)
+    )
+    (pin "1")
+    (pin "2")
+  )
+  (symbol (lib_id "Device:C_Small") (at 138.43 100.33 0) (unit 1)
+    (in_bom yes) (on_board yes) (fields_autoplaced)
+    (property "Reference" "C1" (id 0) (at 140.7541 99.5016 0)
+      (effects (font (size 1.27 1.27)) (justify left))
+    )
+    (property "Value" "10u" (id 1) (at 140.7541 102.0385 0)
+      (effects (font (size 1.27 1.27)) (justify left))
+    )
+    (property "Footprint" "" (id 2) (at 138.43 100.33 0)
+      (effects (font (size 1.27 1.27)) hide)
+    )
+    (property "Datasheet" "~" (id 3) (at 138.43 100.33 0)
+      (effects (font (size 1.27 1.27)) hide)
+    )
+    (pin "1")
+    (pin "2")
+  )
 )

Commit message: WIP update
Parts:
- added C?: 1u, Capacitor_SMD:C_0402_1005Metric, symbol Device:C_Small
- added C?: 10n, Capacitor_SMD:C_0402_1005Metric, symbol Device:C_Small
- added FB?: 600 @ 600 MHz, Inductor_SMD:L_0805_2012Metric, symbol RBoard-rescue:Ferrite_Bead_Small-Device
Connections:
- net GND: now also C?.2, C?.2
- new net +3.3VA: C?.1, C?.1, FB?.1
- new net +3V3: FB?.2
Other:
- note added: "3.3V to 3.3Vfor VDDA"
- note added: "5V to 3.3V"
- moved on the sheet: C1, C2, F1, FB1, U3
