File: Cheap_Shot-Board.kicad_sch (KiCad schematic)
At the start: 1 part

Commit message: WIP update
Other:
- added sheet Connectors (Connectors.kicad_sch)
- added sheet POWER (POWER.kicad_sch)
- note added: "Connectors"
- note added: "POWER"
Changed lines of the file:
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@@
 (kicad_sch (version 20211123) (generator eeschema)
   (paper "A4")
+  (text "Connectors\n" (at 35.56 140.97 0)
+    (effects (font (size 4 4) (thickness 0.8) bold) (justify left bottom))
+  )
+  (text "POWER\n" (at 100.33 140.97 0)
+    (effects (font (size 4 4) (thickness 0.8) bold) (justify left bottom))
+  )
   (symbol (lib_id "MCU_ST_STM32F1:STM32F103C8Tx") (at 106.68 85.09 0) (unit 1)
     (in_bom yes) (on_board yes) (fields_autoplaced)
@@
     (pin "9")
   )
+  (sheet (at 44.45 143.51) (size 24.13 24.13) (fields_autoplaced)
+    (stroke (width 0.1524) (type solid) (color 0 0 0 0))
+    (fill (color 0 0 0 0.0000))
+    (property "Sheet name" "Connectors" (id 0) (at 44.45 142.7984 0)
+      (effects (font (size 1.27 1.27)) (justify left bottom))
+    )
+    (property "Sheet file" "Connectors.kicad_sch" (id 1) (at 44.45 168.2246 0)
+      (effects (font (size 1.27 1.27)) (justify left top))
+    )
+  )
+  (sheet (at 96.52 143.51) (size 24.13 24.13) (fields_autoplaced)
+    (stroke (width 0.1524) (type solid) (color 0 0 0 0))
+    (fill (color 0 0 0 0.0000))
+    (property "Sheet name" "POWER" (id 0) (at 96.52 142.7984 0)
+      (effects (font (size 1.27 1.27)) (justify left bottom))
+    )
+    (property "Sheet file" "POWER.kicad_sch" (id 1) (at 96.52 168.2246 0)
+      (effects (font (size 1.27 1.27)) (justify left top))
+    )
+  )
   (sheet_instances
     (path "/" (page "1"))
+    (path "/64d18fa2-7941-4866-8c1f-29c077bec16a" (page "2"))
+    (path "/9d8a098e-55ac-4559-bb36-a5cce70eb1a0" (page "3"))
   )
   (symbol_instances
+    (path "/64d18fa2-7941-4866-8c1f-29c077bec16a/15d62cba-1c9c-4130-85ae-45ab88c2db85"
+      (reference "#PWR?") (unit 1) (value "+5V") (footprint "")
+    )
+    (path "/64d18fa2-7941-4866-8c1f-29c077bec16a/376d7158-2d3f-4d84-a569-067e8bf210df"
+      (reference "#PWR?") (unit 1) (value "GND") (footprint "")
+    )
+    (path "/64d18fa2-7941-4866-8c1f-29c077bec16a/8ee61d0c-7151-47cb-9687-704e45d7bafc"
+      (reference "#PWR?") (unit 1) (value "+5V") (footprint "")
+    )
+    (path "/64d18fa2-7941-4866-8c1f-29c077bec16a/93696d09-6602-40f5-b39b-1087e979ff10"
+      (reference "#PWR?") (unit 1) (value "GND") (footprint "")
+    )
+    (path "/64d18fa2-7941-4866-8c1f-29c077bec16a/fde43a77-b087-40c9-863f-9197b7567505"
+      (reference "J?") (unit 1) (value "USB_B_Micro") (footprint "")
+    )
+    (path "/9d8a098e-55ac-4559-bb36-a5cce70eb1a0/01ad2c3b-c485-4edd-a4ae-d49717e613df"
+      (reference "U?") (unit 1) (value "XC6206PxxxMR") (footprint "Package_TO_SOT_SMD:SOT-23")
+    )
+    (path "/64d18fa2-7941-4866-8c1f-29c077bec16a/33ea7f72-8d3e-4e3a-919a-48e6a425a45c"
+      (reference "U?") (unit 1) (value "USBLC6-2SC6") (footprint "Package_TO_SOT_SMD:SOT-23-6")
+    )
     (path "/f48efeb8-d579-41e3-a858-bf227dc98d48"
       (reference "U?") (unit 1) (value "STM32F103C8Tx") (footprint "Package_QFP:LQFP-48_7x7mm_P0.5mm")

Commit message: WIP update
Parts:
- gave numbers to parts that had none: 1
Changed lines of the file:
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@@
     (effects (font (size 4 4) (thickness 0.8) bold) (justify left bottom))
+  )
+  (global_label "USB-" (shape input) (at 76.2 96.52 180) (fields_autoplaced)
+    (effects (font (size 1.27 1.27)) (justify right))
+    (property "Intersheet References" "${INTERSHEET_REFS}" (id 0) (at 68.4045 96.5994 0)
+      (effects (font (size 1.27 1.27)) (justify right) hide)
+    )
+  )
+  (global_label "USB+" (shape input) (at 76.2 87.63 180) (fields_autoplaced)
+    (effects (font (size 1.27 1.27)) (justify right))
+    (property "Intersheet References" "${INTERSHEET_REFS}" (id 0) (at 68.4045 87.5506 0)
+      (effects (font (size 1.27 1.27)) (justify right) hide)
+    )
   )
   (symbol (lib_id "MCU_ST_STM32F1:STM32F103C8Tx") (at 106.68 85.09 0) (unit 1)
     (in_bom yes) (on_board yes) (fields_autoplaced)
-    (property "Reference" "U?" (id 0) (at 111.2394 122.6804 0)
+    (property "Reference" "U1" (id 0) (at 111.2394 122.6804 0)
       (effects (font (size 1.27 1.27)) (justify left))
     )
@@
   )
   (symbol_instances
+    (path "/64d18fa2-7941-4866-8c1f-29c077bec16a/93696d09-6602-40f5-b39b-1087e979ff10"
+      (reference "#PWR01") (unit 1) (value "GND") (footprint "")
+    )
+    (path "/64d18fa2-7941-4866-8c1f-29c077bec16a/8ee61d0c-7151-47cb-9687-704e45d7bafc"
+      (reference "#PWR02") (unit 1) (value "+5V") (footprint "")
+    )
     (path "/64d18fa2-7941-4866-8c1f-29c077bec16a/15d62cba-1c9c-4130-85ae-45ab88c2db85"
-      (reference "#PWR?") (unit 1) (value "+5V") (footprint "")
+      (reference "#PWR03") (unit 1) (value "+5V") (footprint "")
     )
     (path "/64d18fa2-7941-4866-8c1f-29c077bec16a/376d7158-2d3f-4d84-a569-067e8bf210df"
-      (reference "#PWR?") (unit 1) (value "GND") (footprint "")
+      (reference "#PWR04") (unit 1) (value "GND") (footprint "")
     )
-    (path "/64d18fa2-7941-4866-8c1f-29c077bec16a/8ee61d0c-7151-47cb-9687-704e45d7bafc"
-      (reference "#PWR?") (unit 1) (value "+5V") (footprint "")
+    (path "/9d8a098e-55ac-4559-bb36-a5cce70eb1a0/a36e1875-ac58-4a47-b8be-9d21a2680e09"
+      (reference "#PWR05") (unit 1) (value "+5V") (footprint "")
     )
-    (path "/64d18fa2-7941-4866-8c1f-29c077bec16a/93696d09-6602-40f5-b39b-1087e979ff10"
-      (reference "#PWR?") (unit 1) (value "GND") (footprint "")
+    (path "/9d8a098e-55ac-4559-bb36-a5cce70eb1a0/ab45534b-b5d9-431d-9156-6c97c198594d"
+      (reference "#PWR06") (unit 1) (value "GND") (footprint "")
+    )
+    (path "/9d8a098e-55ac-4559-bb36-a5cce70eb1a0/951b2b75-08a6-49a4-9765-155650382c3d"
+      (reference "#PWR07") (unit 1) (value "+3.3V") (footprint "")
+    )
+    (path "/9d8a098e-55ac-4559-bb36-a5cce70eb1a0/b8c79952-0449-4a8c-aa4c-5ee7ff5cdd61"
+      (reference "C1") (unit 1) (value "10u") (footprint "")
+    )
+    (path "/9d8a098e-55ac-4559-bb36-a5cce70eb1a0/2bbee2c7-9586-45b9-8348-7c6c6020fc66"
+      (reference "C2") (unit 1) (value "10u") (footprint "")
+    )
+    (path "/9d8a098e-55ac-4559-bb36-a5cce70eb1a0/432a9c48-4be7-4947-a94c-11f212295292"
+      (reference "F1") (unit 1) (value "Fuse") (footprint "")
+    )
+    (path "/9d8a098e-55ac-4559-bb36-a5cce70eb1a0/b4abe4ef-a90e-4a5d-a62d-a56b5c1707fd"
+      (reference "FB1") (unit 1) (value "100@100MHz") (footprint "")
     )
     (path "/64d18fa2-7941-4866-8c1f-29c077bec16a/fde43a77-b087-40c9-863f-9197b7567505"
-      (reference "J?") (unit 1) (value "USB_B_Micro") (footprint "")
+      (reference "J1") (unit 1) (value "USB_B_Micro") (footprint "")
+    )
+    (path "/f48efeb8-d579-41e3-a858-bf227dc98d48"
+      (reference "U1") (unit 1) (value "STM32F103C8Tx") (footprint "Package_QFP:LQFP-48_7x7mm_P0.5mm")
+    )
+    (path "/64d18fa2-7941-4866-8c1f-29c077bec16a/33ea7f72-8d3e-4e3a-919a-48e6a425a45c"
+      (reference "U2") (unit 1) (value "USBLC6-2SC6") (footprint "Package_TO_SOT_SMD:SOT-23-6")
     )
     (path "/9d8a098e-55ac-4559-bb36-a5cce70eb1a0/01ad2c3b-c485-4edd-a4ae-d49717e613df"
-      (reference "U?") (unit 1) (value "XC6206PxxxMR") (footprint "Package_TO_SOT_SMD:SOT-23")
-    )
-    (path "/64d18fa2-7941-4866-8c1f-29c077bec16a/33ea7f72-8d3e-4e3a-919a-48e6a425a45c"
-      (reference "U?") (unit 1) (value "USBLC6-2SC6") (footprint "Package_TO_SOT_SMD:SOT-23-6")
-    )
-    (path "/f48efeb8-d579-41e3-a858-bf227dc98d48"
-      (reference "U?") (unit 1) (value "STM32F103C8Tx") (footprint "Package_QFP:LQFP-48_7x7mm_P0.5mm")
+      (reference "U3") (unit 1) (value "XC6206PxxxMR") (footprint "Package_TO_SOT_SMD:SOT-23")
     )
   )

Commit message: WIP update
Connections:
- net PA0: now reaches U1.10 (PA0)
- net PA1: now reaches U1.11 (PA1)
- net PA2: now reaches U1.12 (PA2)
- net PA3: now reaches U1.13 (PA3)
- net PA4: now reaches U1.14 (PA4)
- net PA5: now reaches U1.15 (PA5)
- net PA6: now reaches U1.16 (PA6)
- net PA7: now reaches U1.17 (PA7)
- net PB0: now reaches U1.18 (PB0)
- net PB1: now reaches U1.19 (PB1)
- net PB2: now reaches U1.20 (PB2)
- net PB10: now reaches U1.21 (PB10)
- net PB11: now reaches U1.22 (PB11)
- net GND: now reaches U1.23 (VSS)
- net GND: now also U1.35 (VSS), U1.47 (VSS), U1.8 (VSSA)
- net +3.3V: now reaches U1.24 (VDD)
- net +3.3V: now also U1.36 (VDD), U1.48 (VDD)
- net PB12: now reaches U1.25 (PB12)
- net PB13: now reaches U1.26 (PB13)
- net PB14: now reaches U1.27 (PB14)
- net PB15: now reaches U1.28 (PB15)
- net PA8: now reaches U1.29 (PA8)
- net PA9: now reaches U1.30 (PA9)
- net PA10: now reaches U1.31 (PA10)
- net PA11: now reaches U1.32 (PA11)
- net PA12: now reaches U1.33 (PA12)
- net PA13: now reaches U1.34 (PA13)
- net PA14: now reaches U1.37 (PA14)
- net PA15: now reaches U1.38 (PA15)
- net PB3: now reaches U1.39 (PB3)
- net PB4: now reaches U1.40 (PB4)
- net PB5: now reaches U1.41 (PB5)
- net PB6: now reaches U1.42 (PB6)
- net PB7: now reaches U1.43 (PB7)
- net BOOT0: now reaches U1.44 (BOOT0)
- net PB8: now reaches U1.45 (PB8)
- net PB9: now reaches U1.46 (PB9)
- net NRST: now reaches U1.7 (NRST)
- net +3.3VA: now reaches U1.9 (VDDA)

Commit message: WIP .sch
Parts:
- added C? (x2): 12p, Capacitor_SMD:C_0402_1005Metric, symbol Device:C_Small
- added D?: RED, LED_SMD:LED_0603_1608Metric, symbol Device:LED_Small
- added R?: 1k, Resistor_SMD:R_0603_1608Metric, symbol Device:R_Small
- added R?: 47, Resistor_SMD:R_0402_1005Metric, symbol Device:R_Small
- added R? (x2): 10k, Resistor_SMD:R_0402_1005Metric, symbol Device:R_Small
- added R? (x2): 2k2, Resistor_SMD:R_0402_1005Metric, symbol Device:R_Small
- added SW?: SW_SPDT, Button_Switch_SMD:SW_SPDT_PCM12, symbol Switch:SW_SPDT
- added Y?: 16MHz, Crystal:Crystal_SMD_3225-4Pin_3.2x2.5mm, symbol Device:Crystal_GND24_Small
Connections:
- net BOOT0: now also R?.2
- net GND: now also C?.2, C?.2, R?.1, R?.2, SW?.3 (C), Y?.2, Y?.4
- new net: D?.1 (K), R?.2
- new net: C?.1, R?.2, Y?.3
- new net: D?.2 (A), R?.1, SW?.2 (B)
- new net +3V3: R?.1, R?.1, SW?.1 (A)
- new net BOOT1: R?.1
- new net HSE_IN: C?.1, Y?.1
- new net HSE_OUT: R?.1
- new net I2C1_SCL: R?.2
- new net I2C1_SDA: R?.2
Other:
- note added: "BOOT0 Switch"
- note added: "HSE"
- note added: "I2C Pull-Ups"
